File: thermalV3_kickad/thermalV3.kicad_pcb (KiCad board)
At the start: 4 copper layers, 90.3 x 94.6 mm, 125 parts, among them J1 cam_brd_top, J2 cam_brd_top, J3 20021321-00020C4LF, P1 battery, P2 button, Q1 STL11N3LLH6, U1 MIMXRT1062DVJ6B, U11 MCP73832T-2DCI/OT, U12 TLV75733PDBVR, U13 STM32F401CBU6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

Commit message: updated pcb footprint
Parts:
- added REF**: CAP1210, AltiumconvertedToKickadPCBfootprints:CAP1210, F.Cu at (132.3, 110.2)
Routing:
- net GND: vias 128 -> 131

Commit message: updated C43 footprint
Parts:
- renumbered REF** to C43
Changed lines of the file:
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@@
 		(at 132.3486 110.2071 90)
 		(descr "Chip Capacitor, 2-Leads, Body 3.20x2.50mm, IPC High Density")
-		(property "Reference" "REF**"
-			(at 0 -2.225 90)
+		(property "Reference" "C43"
+			(at 0 3 90)
 			(layer "F.SilkS")
 			(effects
@@
 		)
 		(property "Value" "CAP1210"
-			(at 0 2.225 90)
+			(at 1.5 3 90)
 			(layer "F.Fab")
+			(hide yes)
 			(effects
 				(font
