File: thermalV3_kickad/sensor board.kicad_sch (KiCad schematic)
At the start: 23 parts, among them J3 20021321-00020C4LF, U14 TLV75528PDBVR, U16 TLV75528PDBVR, U19 Lepton Flir 3.5 sensor, U20 NCP114ASN120T1G, X6 SIT1602BI-13-28E-25.000000

Commit message: project update
Other:
- moved on the sheet: C44, C50, C51, C52, C53, C54, C55, D11, D12B, J3, R26, R27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
